File: ap3722at_mic_breakout/ap3722at_mic_breakout.kicad_pcb (KiCad board)
At the start: 2 copper layers, 20 x 20 mm, 5 parts, among them J1 Conn_01x03_Female, M201 APT3722AT

Commit message: WIP
Other:
- board text added: "V1"
- board text removed: "v1"
Changed lines of the file:
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@@
   (gr_arc (start 161 121) (mid 158.87868 120.12132) (end 158 118) (layer "Edge.Cuts") (width 0.05))
   (gr_line (start 161 101) (end 175 101) (layer "Edge.Cuts") (width 0.05))
+  (gr_text "V1" (at 168 111) (layer "B.SilkS")
+    (effects (font (size 1 1) (thickness 0.15)) (justify mirror))
+  )
   (gr_text "AP3722AT\nMIC" (at 168 103.9) (layer "F.SilkS")
     (effects (font (size 1 1) (thickness 0.15)))
@@
   (gr_text "GND" (at 170.560836 117.20075 90) (layer "F.SilkS")
     (effects (font (size 1 1) (thickness 0.15)) (justify left))
-  )
-  (gr_text "v1" (at 175.1 119.1) (layer "F.SilkS")
-    (effects (font (size 1 1) (thickness 0.15)))
   )
   (segment (start 168.775 108.32) (end 168.775 108) (width 0.25) (layer "F.Cu") (net 1))
@@
     (polygon
       (pts
-        (xy 180 100.074135)
-        (xy 180 122)
-        (xy 156 122)
-        (xy 156 100)
+        (xy 179 100)
+        (xy 179 122)
+        (xy 157 122)
+        (xy 157 100)
       )
     )

Commit message: WIP
Changed lines of the file:
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@@
     (effects (font (size 1 1) (thickness 0.15)) (justify left))
   )
-  (segment (start 168.775 108.32) (end 168.775 108) (width 0.25) (layer "F.Cu") (net 1))
   (segment (start 169.33 111.575) (end 170.175 111.575) (width 0.25) (layer "F.Cu") (net 1))
   (segment (start 169.33 110.425) (end 170.175 110.425) (width 0.25) (layer "F.Cu") (net 1))

Commit message: final touches + v1 jlcpcb fab files
Parts:
- moved REF** 16.3 mm to (158.9, 120.1), turned to 90 degrees
- moved REF** 16.3 mm to (158.9, 105.9), turned to 90 degrees
- moved J1 9.21 mm to (174.0, 115.5), turned to 180 degrees
- moved C201 7.07 mm to (163.0, 113.0), turned to -90 degrees
- moved M201 2.83 mm to (166.0, 113.0), turned to 180 degrees
