File: wm8758b_codec_breakout/wm8758b_codec_breakout.kicad_pcb (KiCad board)
At the start: 2 copper layers, 40 x 40 mm, 21 parts, among them J1 Conn_01x12, J101 AudioJack3, J102 AudioJack3, J2 Conn_01x12, U1 WM8758B

Commit message: WIP
Parts:
- moved C6 22.8 mm to (144.6, 70.1), turned to 180 degrees
- moved C2 20.2 mm to (156.2, 72.5)
- moved C5 20.2 mm to (154.6, 72.5)
- moved C1 20.1 mm to (149.0, 72.5)
- moved C11 20.1 mm to (144.6, 78.1)
- moved C12 20.1 mm to (155.4, 79.3)
- moved C16 20.1 mm to (144.6, 73.3)
- moved U1 20.1 mm to (150.0, 77.3)
- moved C10 20.1 mm to (144.6, 74.9)
- moved C13 20.1 mm to (155.4, 77.7)
- moved C15 20.1 mm to (144.6, 71.7)
- moved C19 20.1 mm to (144.6, 76.5)
- moved C8 20.1 mm to (144.6, 79.7)
- moved REF** 20.0 mm to (167.0, 63.0)
- moved REF** 20.0 mm to (133.0, 63.0)
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Routing:
- net VDD: track 0.00 -> 57.7 mm, vias 0 -> 3
- net MICBIAS: track 0.00 -> 31.0 mm
- net MCLK: track 0.00 -> 23.4 mm
- net CSB_GPIO1: track 0.00 -> 22.5 mm
- net DACDAT: track 0.00 -> 21.8 mm
- net LOUT1: track 0.00 -> 21.4 mm
- net ROUT1: track 0.00 -> 20.9 mm
- net SCLK: track 0.00 -> 20.7 mm
- net ADCDAT: track 0.00 -> 20.1 mm
- net SDIN: track 0.00 -> 19.3 mm
- net BCLK: track 0.00 -> 19.0 mm
- net MODE: track 0.00 -> 18.5 mm
- net OUT4: track 0.00 -> 18.2 mm
- net LRC: track 0.00 -> 17.8 mm
- net OUT3: track 0.00 -> 17.3 mm
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Other:
- board text added: "CSB"
- board text added: "V1"
- board text removed: "CSB/GPIO1"

Commit message: WIP
Parts:
- moved J101 12.1 mm to (144.0, 99.9)
- moved J102 12.0 mm to (156.0, 99.9)
Connections:
- J101 pad R: unconnected-(J101-PadR) -> RIN
- J101 pad T: unconnected-(J101-PadT) -> LIN
- J102 pad R: unconnected-(J102-PadR) -> ROUT1
- J102 pad T: unconnected-(J102-PadT) -> LOUT1
Routing:
- net ROUT1: track 20.9 -> 56.9 mm, vias 0 -> 2
- net LIN: track 12.8 -> 42.9 mm, vias 0 -> 2
- net LOUT1: track 21.4 -> 47.2 mm, vias 0 -> 2
- net RIN: track 11.6 -> 30.9 mm, vias 0 -> 2
Other:
- board text added: "HP"
- board text added: "MIC"

Commit message: final touches + v1 jlcpcb fab files
Routing:
- net GND: track 4.58 -> 20.3 mm, vias 2 -> 11
- net ROUT1: track 56.9 -> 57.9 mm
Changed lines of the file:
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@@
       (drillshape 0)
       (scaleselection 1)
-      (outputdirectory "order/1.0/")
+      (outputdirectory "fab/v1/jlcpcb")
     )
   )
@@
   )
   (segment (start 152.3 75.55) (end 152.35 75.55) (width 0.25) (layer "F.Cu") (net 1))
+  (segment (start 149 71.6) (end 150.4 70.2) (width 0.25) (layer "F.Cu") (net 1))
   (segment (start 149.75 78.775) (end 149.56875 78.59375) (width 0.25) (layer "F.Cu") (net 1))
   (segment (start 149.75 79.6) (end 149.75 78.775) (width 0.25) (layer "F.Cu") (net 1))
+  (segment (start 154.6 70.8) (end 155 70.4) (width 0.25) (layer "F.Cu") (net 1))
+  (segment (start 156.175 77.7) (end 157.3 77.7) (width 0.25) (layer "F.Cu") (net 1))
+  (segment (start 149.225 83.6) (end 149.225 84.975) (width 0.25) (layer "F.Cu") (net 1))
+  (segment (start 143.825 70.1) (end 142.7 70.1) (width 0.25) (layer "F.Cu") (net 1))
+  (segment (start 156.2 70.6) (end 156.4 70.4) (width 0.25) (layer "F.Cu") (net 1))
+  (segment (start 147.75 97.8) (end 147.75 96.45) (width 0.25) (layer "F.Cu") (net 1))
+  (segment (start 157.3 79.3) (end 157.4 79.2) (width 0.25) (layer "F.Cu") (net 1))
+  (segment (start 142.7 70.1) (end 142.6 70) (width 0.25) (layer "F.Cu") (net 1))
   (segment (start 149.75 79.6) (end 149.75 80.55) (width 0.25) (layer "F.Cu") (net 1))
+  (segment (start 159.75 97.8) (end 162.2 97.8) (width 0.25) (layer "F.Cu") (net 1))
   (segment (start 152.35 75.55) (end 153.1 74.8) (width 0.25) (layer "F.Cu") (net 1))
+  (segment (start 149.225 84.975) (end 149.2 85) (width 0.25) (layer "F.Cu") (net 1))
   (segment (start 149.75 80.55) (end 150 80.8) (width 0.25) (layer "F.Cu") (net 1))
+  (segment (start 147.75 96.45) (end 147.8 96.4) (width 0.25) (layer "F.Cu") (net 1))
+  (segment (start 156.2 71.725) (end 156.2 70.6) (width 0.25) (layer "F.Cu") (net 1))
   (segment (start 150.25 75) (end 150.25 75.825) (width 0.25) (layer "F.Cu") (net 1))
+  (segment (start 154.6 71.725) (end 154.6 70.8) (width 0.25) (layer "F.Cu") (net 1))
+  (segment (start 149.225 82) (end 149.225 83.6) (width 0.25) (layer "F.Cu") (net 1))
+  (segment (start 149 71.725) (end 149 71.6) (width 0.25) (layer "F.Cu") (net 1))
+  (segment (start 157.3 77.7) (end 157.4 77.8) (width 0.25) (layer "F.Cu") (net 1))
+  (segment (start 156.175 79.3) (end 157.3 79.3) (width 0.25) (layer "F.Cu") (net 1))
   (segment (start 150.25 75.825) (end 150.43125 76.00625) (width 0.25) (layer "F.Cu") (net 1))
+  (via (at 156.4 70.4) (size 0.8) (drill 0.4) (layers "F.Cu" "B.Cu") (net 1))
   (via (at 150 80.8) (size 0.8) (drill 0.4) (layers "F.Cu" "B.Cu") (net 1))
   (via (at 153.1 74.8) (size 0.8) (drill 0.4) (layers "F.Cu" "B.Cu") (net 1))
+  (via (at 162.2 97.8) (size 0.8) (drill 0.4) (layers "F.Cu" "B.Cu") (net 1))
+  (via (at 142.6 70) (size 0.8) (drill 0.4) (layers "F.Cu" "B.Cu") (net 1))
+  (via (at 157.4 77.8) (size 0.8) (drill 0.4) (layers "F.Cu" "B.Cu") (net 1))
+  (via (at 157.4 79.2) (size 0.8) (drill 0.4) (layers "F.Cu" "B.Cu") (net 1))
+  (via (at 150.4 70.2) (size 0.8) (drill 0.4) (layers "F.Cu" "B.Cu") (net 1))
+  (via (at 147.8 96.4) (size 0.8) (drill 0.4) (layers "F.Cu" "B.Cu") (net 1))
+  (via (at 155 70.4) (size 0.8) (drill 0.4) (layers "F.Cu" "B.Cu") (net 1))
+  (via (at 149.2 85) (size 0.8) (drill 0.4) (layers "F.Cu" "B.Cu") (net 1))
   (segment (start 153.69885 73.625988) (end 154.122382 74.04952) (width 0.25) (layer "F.Cu") (net 2))
   (segment (start 159.876477 94.275499) (end 166.119499 94.275499) (width 0.25) (layer "F.Cu") (net 2))
@@
   (segment (start 133.796 67.996) (end 137.6 71.8) (width 0.2) (layer "F.Cu") (net 15))
   (segment (start 143.725 71.8) (end 143.825 71.7) (width 0.2) (layer "F.Cu") (net 15))
-  (segment (start 166.93 69.686) (end 167.78 70.536) (width 0.25) (layer "F.Cu") (net 16))
+  (segment (start 159.7 89.6) (end 159.8 89.5) (width 0.25) (layer "F.Cu") (net 16))
   (segment (start 149.25 75) (end 149.25 74.415274) (width 0.25) (layer "F.Cu") (net 16))
-  (segment (start 153.979274 69.686) (end 166.93 69.686) (width 0.25) (layer "F.Cu") (net 16))
-  (segment (start 159.7 89.6) (end 159.8 89.5) (width 0.25) (layer "F.Cu") (net 16))
   (segment (start 159.7 91.05) (end 159.7 89.6) (width 0.25) (layer "F.Cu") (net 16))
   (segment (start 165.4 71.9) (end 166.416 71.9) (width 0.25) (layer "F.Cu") (net 16))
+  (segment (start 149.25 74.415274) (end 154.439285 69.225989) (width 0.25) (layer "F.Cu") (net 16))
   (segment (start 166.416 71.9) (end 167.78 70.536) (width 0.25) (layer "F.Cu") (net 16))
-  (segment (start 149.25 74.415274) (end 153.979274 69.686) (width 0.25) (layer "F.Cu") (net 16))
+  (segment (start 154.439285 69.225989) (end 166.469989 69.225989) (width 0.25) (layer "F.Cu") (net 16))
+  (segment (start 166.469989 69.225989) (end 167.78 70.536) (width 0.25) (layer "F.Cu") (net 16))
   (via (at 159.8 89.5) (size 0.8) (drill 0.4) (layers "F.Cu" "B.Cu") (net 16))
   (via (at 165.4 71.9) (size 0.8) (drill 0.4) (layers "F.Cu" "B.Cu") (net 16))
@@
   (segment (start 163.2 71.9) (end 159.8 75.3) (width 0.25) (layer "B.Cu") (net 16))
   (segment (start 165.4 71.9) (end 163.2 71.9) (width 0.25) (layer "B.Cu") (net 16))
-  (segment (start 149.75 74.550978) (end 153.350498 70.95048) (width 0.25) (layer "F.Cu") (net 17))
-  (segment (start 162.05048 70.95048) (end 164.176 73.076) (width 0.25) (layer "F.Cu") (net 17))
-  (segment (start 153.350498 70.95048) (end 162.05048 70.95048) (width 0.25) (layer "F.Cu") (net 17))
+  (segment (start 154.699901 69.675499) (end 160.775499 69.675499) (width 0.25) (layer "F.Cu") (net 17))
+  (segment (start 160.775499 69.675499) (end 164.176 73.076) (width 0.25) (layer "F.Cu") (net 17))
   (segment (start 164.176 73.076) (end 167.78 73.076) (width 0.25) (layer "F.Cu") (net 17))
-  (segment (start 149.75 75) (end 149.75 74.550978) (width 0.25) (layer "F.Cu") (net 17))
   (segment (start 152.25 95.8) (end 163 95.8) (width 0.25) (layer "F.Cu") (net 17))
+  (segment (start 149.75 75) (end 149.75 74.6254) (width 0.25) (layer "F.Cu") (net 17))
+  (segment (start 149.75 74.6254) (end 154.699901 69.675499) (width 0.25) (layer "F.Cu") (net 17))
   (segment (start 165.2 74.6) (end 166.256 74.6) (width 0.25) (layer "F.Cu") (net 17))
   (segment (start 166.256 74.6) (end 167.78 73.076) (width 0.25) (layer "F.Cu") (net 17))
@@
   (segment (start 146.42957 78.1) (end 146.97957 77.55) (width 0.25) (layer "F.Cu") (net 30))
   (segment (start 147.7 75.55) (end 146.60048 74.45048) (width 0.25) (layer "F.Cu") (net 31))
+  (segment (start 145.375 71.7) (end 146.60048 72.92548) (width 0.25) (layer "F.Cu") (net 31))
   (segment (start 146.60048 74.45048) (end 146.60048 72.92548) (width 0.25) (layer "F.Cu") (net 31))
-  (segment (start 145.375 71.7) (end 145.375 71.902138) (width 0.25) (layer "F.Cu") (net 31))
-  (segment (start 146.60048 72.92548) (end 145.375 71.7) (width 0.25) (layer "F.Cu") (net 31))
   (segment (start 146.14952 74.948542) (end 147.250978 76.05) (width 0.25) (layer "F.Cu") (net 32))
   (segment (start 146.14952 74.07452) (end 146.14952 74.948542) (width 0.25) (layer "F.Cu") (net 32))
