File: wm8758b_codec_breakout/wm8758b_codec_breakout.kicad_sch (KiCad schematic)
At the start: 19 parts, among them J1 Conn_01x12, J2 Conn_01x12, U1 WM8758B

Commit message: WIP
Parts:
- gave numbers to parts that had none: 2
Changed lines of the file:
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@@
   (symbol (lib_id "Connector:AudioJack3") (at 181.61 59.69 0) (unit 1)
     (in_bom yes) (on_board yes) (fields_autoplaced)
-    (property "Reference" "J?" (id 0) (at 179.705 50.8 0))
+    (property "Reference" "J102" (id 0) (at 179.705 50.8 0))
     (property "Value" "AudioJack3" (id 1) (at 179.705 53.34 0))
     (property "Footprint" "WM8758B_breakout:PJ-320B-3A" (id 2) (at 181.61 59.69 0)
@@
   (symbol (lib_id "Connector:AudioJack3") (at 181.61 41.91 0) (unit 1)
     (in_bom yes) (on_board yes) (fields_autoplaced)
-    (property "Reference" "J?" (id 0) (at 179.705 33.02 0))
+    (property "Reference" "J101" (id 0) (at 179.705 33.02 0))
     (property "Value" "AudioJack3" (id 1) (at 179.705 35.56 0))
     (property "Footprint" "WM8758B_breakout:PJ-320B-3A" (id 2) (at 181.61 41.91 0)
@@
       (reference "J2") (unit 1) (value "Conn_01x12") (footprint "Connector_PinSocket_2.54mm:PinSocket_1x12_P2.54mm_Vertical")
     )
+    (path "/e6e48900-5e32-4819-b8bb-9070db430e97"
+      (reference "J101") (unit 1) (value "AudioJack3") (footprint "WM8758B_breakout:PJ-320B-3A")
+    )
     (path "/a8962eda-0d23-4bc3-8c77-e73285b2c80e"
-      (reference "J?") (unit 1) (value "AudioJack3") (footprint "WM8758B_breakout:PJ-320B-3A")
-    )
-    (path "/e6e48900-5e32-4819-b8bb-9070db430e97"
-      (reference "J?") (unit 1) (value "AudioJack3") (footprint "WM8758B_breakout:PJ-320B-3A")
+      (reference "J102") (unit 1) (value "AudioJack3") (footprint "WM8758B_breakout:PJ-320B-3A")
     )
     (path "/00000000-0000-0000-0000-000061297471"

Commit message: WIP
Connections:
- net LIN: now also J101.T
- net LOUT1: now also J102.T
- net RIN: now also J101.R
- net ROUT1: now also J102.R
Changed lines of the file:
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@@
+    )
+  )
+  (global_label "ROUT1" (shape input) (at 186.69 59.69 0) (fields_autoplaced)
+    (effects (font (size 1.27 1.27)) (justify left))
+    (property "Intersheet References" "${INTERSHEET_REFS}" (id 0) (at 309.88 156.21 0)
+      (effects (font (size 1.27 1.27)) hide)
     )
   )
@@
     )
   )
+  (global_label "RIN" (shape input) (at 186.69 41.91 0) (fields_autoplaced)
+    (effects (font (size 1.27 1.27)) (justify left))
+    (property "Intersheet References" "${INTERSHEET_REFS}" (id 0) (at 11.43 -88.9 0)
+      (effects (font (size 1.27 1.27)) hide)
+    )
+  )
   (global_label "RIP" (shape input) (at 175.26 140.97 0) (fields_autoplaced)
     (effects (font (size 1.27 1.27)) (justify left))
@@
     )
   )
+  (global_label "LOUT1" (shape input) (at 186.69 62.23 0) (fields_autoplaced)
+    (effects (font (size 1.27 1.27)) (justify left))
+    (property "Intersheet References" "${INTERSHEET_REFS}" (id 0) (at 309.88 161.29 0)
+      (effects (font (size 1.27 1.27)) hide)
+    )
+  )
   (global_label "OUT3" (shape input) (at 147.32 35.56 270) (fields_autoplaced)
     (effects (font (size 1.27 1.27)) (justify right))
@@
       (effects (font (size 1.27 1.27)) hide)
     )
+  )
+  (global_label "LIN" (shape input) (at 186.69 44.45 0) (fields_autoplaced)
+    (effects (font (size 1.27 1.27)) (justify left))
+    (property "Intersheet References" "${INTERSHEET_REFS}" (id 0) (at 300.99 187.96 0)
+      (effects (font (size 1.27 1.27)) hide)
+    )

Commit message: final touches + v1 jlcpcb fab files
Parts:
- J101, J102: LCSC Part (none) -> C707224; MSCS Part C707224 -> (none)
Changed lines of the file:
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@@
       (effects (font (size 1.27 1.27)) hide)
     )
-    (property "MSCS Part" "C707224" (id 4) (at 181.61 59.69 0)
+    (property "LCSC Part" "C707224" (id 4) (at 181.61 59.69 0)
       (effects (font (size 1.27 1.27)) hide)
     )
@@
       (effects (font (size 1.27 1.27)) hide)
     )
-    (property "MSCS Part" "C707224" (id 4) (at 181.61 41.91 0)
+    (property "LCSC Part" "C707224" (id 4) (at 181.61 41.91 0)
       (effects (font (size 1.27 1.27)) hide)
     )
