File: wm8904_codec_breakout/wm8904_codec_breakout.kicad_pcb (KiCad board)
At the start: 2 copper layers, 40 x 40 mm, 30 parts, among them J101 Conn_01x12_Female, J102 Conn_01x12_Female, J103 AudioJack3, J104 AudioJack3, U101 AMS1117-1.8, U201 wm8904

Commit message: WIP
Parts:
- added TP101: 1V8, TestPoint:TestPoint_Pad_D1.5mm, F.Cu at (156.6, 80.4)
- added TP102: GND, TestPoint:TestPoint_Pad_D1.5mm, F.Cu at (156.6, 84.4)
- moved U101 15.0 mm to (150.0, 82.4)
- moved J103 12.2 mm to (144.0, 99.9)
- moved J104 12.1 mm to (156.0, 99.9)
- moved C212 7.24 mm to (145.8, 68.2)
- moved C214 7.24 mm to (146.8, 68.2)
- moved C215 6.93 mm to (150.6, 68.2)
- moved C216 6.93 mm to (149.6, 68.2)
- moved C213 6.93 mm to (151.6, 68.2)
- moved R203 6.48 mm to (144.0, 72.2), turned to 180 degrees
- moved C201 5.80 mm to (149.8, 77.5)
- moved C202 5.80 mm to (147.8, 77.5)
- moved C203 5.80 mm to (150.8, 77.5)
- moved C204 5.80 mm to (152.3, 77.1)
- moved U201 5.80 mm to (150.0, 73.2)
- moved R205 5.55 mm to (148.6, 68.2), turned to -90 degrees
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Routing:
- net IN2R: track 0.00 -> 50.2 mm, vias 0 -> 2
- net HPOUTR: track 0.00 -> 47.5 mm, vias 0 -> 2
- net 1V8: track 0.00 -> 41.1 mm, vias 0 -> 3
- net HPOUTL: track 0.00 -> 35.3 mm, vias 0 -> 2
- net IN2L: track 0.00 -> 34.0 mm, vias 0 -> 2
- net SCLK: track 0.00 -> 29.5 mm
- net SDA: track 0.00 -> 27.0 mm
- net GND: track 0.00 -> 25.9 mm, vias 0 -> 16
- net IRQ/GPIO1: track 0.00 -> 22.9 mm
- net DACDAT: track 0.00 -> 21.7 mm
- net LINEOUTR: track 0.00 -> 21.3 mm
- net VDD: track 0.00 -> 20.9 mm
- net ADCDAT: track 0.00 -> 20.8 mm
- net LRCLK: track 0.00 -> 19.9 mm
- net BCLK/GPIO4: track 0.00 -> 19.0 mm
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Other:
- board text added: "IRQ"
- board text removed: "IRQ/GPIO1"

Commit message: WIP
Other:
- board text added: "HP"
- board text added: "MIC"
- board text removed: "HPOUT"
- board text removed: "IN2"
Changed lines of the file:
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@@
     (effects (font (size 1 1) (thickness 0.15)) (justify left))
   )
-  (gr_text "HPOUT" (at 156 87.4) (layer "F.SilkS")
+  (gr_text "HP" (at 156 87.6) (layer "F.SilkS")
     (effects (font (size 1 1) (thickness 0.15)))
   )
@@
     (effects (font (size 1 1) (thickness 0.15)) (justify right))
   )
-  (gr_text "IN2" (at 144 87.4) (layer "F.SilkS")
+  (gr_text "MIC" (at 144 87.6) (layer "F.SilkS")
     (effects (font (size 1 1) (thickness 0.15)))
   )

Commit message: final touches + v1 jlcpcb fab files
Parts:
- removed TP101: 1V8, TestPoint:TestPoint_Pad_D1.5mm
- removed TP102: GND, TestPoint:TestPoint_Pad_D1.5mm
- moved C204 0.86 mm to (152.3, 76.2)
Connections:
- J101 pad 12: VDD -> 1V8
Routing:
- net 1V8: track 41.1 -> 67.6 mm
- net VDD: track 20.9 -> 18.3 mm
- net GND: track 25.9 -> 24.0 mm, vias 16 -> 15
- net Net-(C204-Pad2): track 3.45 -> 2.59 mm
- net Net-(C204-Pad1): track 2.25 -> 1.39 mm
Other:
- board text added: "1V8"
